File: Hardware/qwiic_blower.brd (EAGLE design)
At the start: 152.7 x 152.4 mm, 318 parts, among them J1 QWIIC_RIGHT_ANGLE, J11 QWIIC_RIGHT_ANGLE, J12 QWIIC_RIGHT_ANGLE, J13 AVR_SPI_PROG_3X2NS, J16 QWIIC_RIGHT_ANGLE, J17 QWIIC_RIGHT_ANGLE, J18 AVR_SPI_PROG_3X2NS, J2 QWIIC_RIGHT_ANGLE, J21 QWIIC_RIGHT_ANGLE, J22 QWIIC_RIGHT_ANGLE, J23 AVR_SPI_PROG_3X2NS, J26 QWIIC_RIGHT_ANGLE, J27 QWIIC_RIGHT_ANGLE, J28 AVR_SPI_PROG_3X2NS, J3 AVR_SPI_PROG_3X2NS, J6 QWIIC_RIGHT_ANGLE, J7 QWIIC_RIGHT_ANGLE, J8 AVR_SPI_PROG_3X2NS, Q1 310mA/60V/1.6Ω, Q10 310mA/60V/1.6Ω, Q11 310mA/60V/1.6Ω, Q12 310mA/60V/1.6Ω, Q2 310mA/60V/1.6Ω, Q3 310mA/60V/1.6Ω, Q4 310mA/60V/1.6Ω, Q5 310mA/60V/1.6Ω, Q6 310mA/60V/1.6Ω, Q7 310mA/60V/1.6Ω, Q8 310mA/60V/1.6Ω, Q9 310mA/60V/1.6Ω, U1 ATtiny841, U10 ATtiny841, U11 PAM2401, U12 ATtiny841, U2 PAM2401, U3 PAM2401, U4 ATtiny841, U5 PAM2401, U6 ATtiny841, U7 PAM2401, U8 ATtiny841, U9 PAM2401, Y1 16MHz, Y2 16MHz, Y3 16MHz, Y4 16MHz, Y5 16MHz, Y6 16MHz

Commit message: V1 Docs and Housecleaning
Parts:
- removed C10, C11, C17, C18, C24, C25, C31, C32, C38, C39: 0.1uF, SparkFun-Capacitors:0603
- removed C12, C19, C26, C33, C40: 1.0uF, SparkFun-Capacitors:0603
- removed C13, C14, C20, C21, C27, C28, C34, C35, C41, C42: 22pF, SparkFun-Capacitors:0603
- removed C15, C22, C29, C36, C8: 10uF, SparkFun-Capacitors:0603
- removed C16, C23, C30, C37, C9: 22uF, SparkFun-Capacitors:0805
- removed D2, D3, D4, D5, D6: RED, SparkFun-LED:LED-0603
- removed E$1, E$2, E$3, E$4: (no value), SparkFun-Aesthetics:FIDUCIAL-1X2
- removed E$5, E$6: (no value), SparkFun-Retired:FIDUCIAL-1.5X3
- removed H10, H11, H12, H13, H14, H15, H16, H17, H18, H19, H20, H21, H22, H23, H24, H5, H6, H7, H8, H9: STAND-OFF, SparkFun-Hardware:STAND-OFF
- removed J10, J15, J20, J25, J30: (no value), SparkFun-Connectors:1X02_NO_SILK
- removed J11, J12, J16, J17, J21, J22, J26, J27, J6, J7: QWIIC_RIGHT_ANGLE, SparkFun-Connectors:JST04_1MM_RA
- removed J13, J18, J23, J28, J8: AVR_SPI_PROG_3X2NS, SparkFun-Connectors:2X3-NS
- removed J14, J19, J24, J29, J9: (no value), SparkFun-Connectors:1X04_NO_SILK
- removed L2, L3, L4, L5, L6: 2.2μH, SparkFun-Coils:0806
- removed Q1, Q10, Q11, Q12, Q4, Q5, Q6, Q7, Q8, Q9: 310mA/60V/1.6Ω, SparkFun-DiscreteSemi:SOT323
- removed R10, R12, R14, R19, R20, R21, R22, R27, R28, R29, R30, R35, R36, R37, R38, R43, R44, R45, R46, R9: 2.2k, SparkFun-Resistors:0603
- removed R15, R23, R31, R39, R47: 10k, SparkFun-Resistors:0603
- removed R16, R24, R32, R40, R48: 1k, SparkFun-Resistors:0603
- removed R17, R25, R33, R41, R7: 750K, SparkFun-Resistors:0603
- removed R18, R26, R34, R42, R8: 100k, SparkFun-Resistors:0603
- removed U$100, U$121, U$37, U$58, U$79: (no value), output:AIR_BLOWS_OUT_THIS_WAY0
- removed U$101, U$122, U$38, U$59, U$80: (no value), output:_QWIIC_BLOWER_0
- removed U$102, U$123, U$39, U$60, U$81: (no value), SparkX:SPARKX-LARGE
- removed U$103, U$124, U$40, U$61, U$82: NINTENDO_SWITCH_FAN, SparkFun-Connectors:FPC_4_0.5MM
- removed U$104, U$125, U$41, U$62, U$83: (no value), SparkFun-Aesthetics:OSHW-LOGO-S
- removed U$105, U$126, U$42, U$63, U$84: (no value), output:PWR0
- removed U$106, U$22, U$43, U$64, U$85: (no value), output:#_TACH#0
- removed U$107, U$23, U$44, U$65, U$86: (no value), output:#_PWM#0
- removed U$108, U$24, U$45, U$66, U$87: (no value), output:#_GND#0
- removed U$109, U$25, U$46, U$67, U$88: (no value), output:#_3#3V#0
- removed U$110, U$26, U$47, U$68, U$89: (no value), output:#_SDA#0
- removed U$111, U$27, U$48, U$69, U$90: (no value), output:#_SCL#0
- removed U$112, U$28, U$49, U$70, U$91: (no value), output:#SCL_#0
- removed U$113, U$29, U$50, U$71, U$92: (no value), output:#SDA_#0
- removed U$114, U$30, U$51, U$72, U$93: (no value), output:#3#3V_#0
- removed U$115, U$31, U$52, U$73, U$94: (no value), output:#GND_#0
- removed U$116, U$32, U$53, U$74, U$95: (no value), output:#PWM_#0
- removed U$117, U$33, U$54, U$75, U$96: (no value), output:#TACH_#0
- removed U$118, U$34, U$55, U$76, U$97: (no value), SparkFun-Aesthetics:QWIIC_4MM
- removed U$119, U$35, U$56, U$77, U$98: (no value), output:QWIIC_BLOWER0
- removed U$120, U$36, U$57, U$78, U$99: (no value), SparkX:SPARKX-TINY
- removed U10, U12, U4, U6, U8: ATtiny841, SparkFun-IC-Microcontroller:SO14
- removed U11, U2, U5, U7, U9: PAM2401, SparkFun-IC-Power:MSOP8
- removed Y1, Y3, Y4, Y5, Y6: 16MHz, SparkFun-Clocks:CRYSTAL-SMD-2.0X1.6MM
- added FRAME1: FRAME-LETTER, SparkFun-Aesthetics:CREATIVE_COMMONS
Connections:
- removed net !RST1: J8.5, R15.1, U4.4
- removed net !RST2: J13.5, R23.1, U6.4
- removed net !RST3: J18.5, R31.1, U8.4
- removed net !RST4: J23.5, R39.1, U10.4
- removed net !RST5: J28.5, R47.1, U12.4
- removed net 25KHZ_PWM1: J10.2, U$40.4, U4.10
- removed net 25KHZ_PWM2: J15.2, U$61.4, U6.10
- removed net 25KHZ_PWM3: J20.2, U$82.4, U8.10
- removed net 25KHZ_PWM4: J25.2, U$103.4, U10.10
- removed net 25KHZ_PWM5: J30.2, U$124.4, U12.10
- removed net 3.3V1: C8.1, J6.2, J7.2, J9.2, L2.1, Q1.1, Q4.1, R12.2, R9.2, U2.2, U2.3
- removed net 3.3V2: C15.1, J11.2, J12.2, J14.2, L3.1, Q5.1, Q6.1, R19.2, R21.2, U5.2, U5.3
- removed net 3.3V3: C22.1, J16.2, J17.2, J19.2, L4.1, Q7.1, Q8.1, R27.2, R29.2, U7.2, U7.3
- removed net 3.3V4: C29.1, J21.2, J22.2, J24.2, L5.1, Q10.1, Q9.1, R35.2, R37.2, U9.2, U9.3
- removed net 3.3V5: C36.1, J26.2, J27.2, J29.2, L6.1, Q11.1, Q12.1, R43.2, R45.2, U11.2, U11.3
- removed net 5V1: C10.1, C11.1, C12.1, C9.1, D2.A, J8.2, R10.2, R14.2, R15.2, R7.2, U$40.1, U2.7, U4.1
- removed net 5V2: C16.1, C17.1, C18.1, C19.1, D3.A, J13.2, R17.2, R20.2, R22.2, R23.2, U$61.1, U5.7, U6.1
- removed net 5V3: C23.1, C24.1, C25.1, C26.1, D4.A, J18.2, R25.2, R28.2, R30.2, R31.2, U$82.1, U7.7, U8.1
- removed net 5V4: C30.1, C31.1, C32.1, C33.1, D5.A, J23.2, R33.2, R36.2, R38.2, R39.2, U$103.1, U10.1, U9.7
- removed net 5V5: C37.1, C38.1, C39.1, C40.1, D6.A, J28.2, R41.2, R44.2, R46.2, R47.2, U$124.1, U11.7, U12.1
- removed net CIPO1: J8.1, U4.8
- removed net CIPO2: J13.1, U6.8
- removed net CIPO3: J18.1, U8.8
- removed net CIPO4: J23.1, U10.8
- removed net CIPO5: J28.1, U12.8
- removed net FAN_TACH1: J10.1, U$40.2, U4.6
- removed net FAN_TACH2: J15.1, U$61.2, U6.6
- removed net FAN_TACH3: J20.1, U$82.2, U8.6
- removed net FAN_TACH4: J25.1, U$103.2, U10.6
- removed net FAN_TACH5: J30.1, U$124.2, U12.6
- removed net GND1: C10.2, C11.2, C12.2, C13.1, C14.1, C8.2, C9.2, J6.1, J7.1, J8.6, J9.1, R16.1, R8.1, U$40.3, U2.4, U2.8, U4.14
- removed net GND2: C15.2, C16.2, C17.2, C18.2, C19.2, C20.1, C21.1, J11.1, J12.1, J13.6, J14.1, R18.1, R24.1, U$61.3, U5.4, U5.8, U6.14
- removed net GND3: C22.2, C23.2, C24.2, C25.2, C26.2, C27.1, C28.1, J16.1, J17.1, J18.6, J19.1, R26.1, R32.1, U$82.3, U7.4, U7.8, U8.14
- removed net GND4: C29.2, C30.2, C31.2, C32.2, C33.2, C34.1, C35.1, J21.1, J22.1, J23.6, J24.1, R34.1, R40.1, U$103.3, U10.14, U9.4, U9.8
- removed net GND5: C36.2, C37.2, C38.2, C39.2, C40.2, C41.1, C42.1, J26.1, J27.1, J28.6, J29.1, R42.1, R48.1, U$124.3, U11.4, U11.8, U12.14
- removed net HV_SCL1: J8.3, Q1.3, R10.1, U4.9
- removed net HV_SCL2: J13.3, Q5.3, R20.1, U6.9
- removed net HV_SCL3: J18.3, Q7.3, R28.1, U8.9
- removed net HV_SCL4: J23.3, Q9.3, R36.1, U10.9
- removed net HV_SCL5: J28.3, Q11.3, R44.1, U12.9
- removed net HV_SDA1: J8.4, Q4.3, R14.1, U4.7
- removed net HV_SDA2: J13.4, Q6.3, R22.1, U6.7
- removed net HV_SDA3: J18.4, Q8.3, R30.1, U8.7
- removed net HV_SDA4: J23.4, Q10.3, R38.1, U10.7
- removed net HV_SDA5: J28.4, Q12.3, R46.1, U12.7
- removed net N$10: D2.C, R16.2
- removed net N$11: R17.1, R18.2, U5.5
- removed net N$12: L3.2, U5.1
- removed net N$13: C21.2, U6.3, Y3.1
- removed net N$14: C20.2, U6.2, Y3.3
- removed net N$15: D3.C, R24.2
- removed net N$16: R25.1, R26.2, U7.5
- removed net N$17: L4.2, U7.1
- removed net N$18: C28.2, U8.3, Y4.1
- removed net N$19: C27.2, U8.2, Y4.3
- removed net N$20: D4.C, R32.2
- removed net N$21: R33.1, R34.2, U9.5
- removed net N$22: L5.2, U9.1
- removed net N$23: C35.2, U10.3, Y5.1
- removed net N$24: C34.2, U10.2, Y5.3
- removed net N$25: D5.C, R40.2
- removed net N$26: R41.1, R42.2, U11.5
- removed net N$27: L6.2, U11.1
- removed net N$28: C42.2, U12.3, Y6.1
- removed net N$29: C41.2, U12.2, Y6.3
- removed net N$30: D6.C, R48.2
- removed net N$6: R7.1, R8.2, U2.5
- removed net N$7: L2.2, U2.1
- removed net N$8: C14.2, U4.3, Y1.1
- removed net N$9: C13.2, U4.2, Y1.3
- removed net SCL1: J6.4, J7.4, J9.4, Q1.2, R9.1
- removed net SCL2: J11.4, J12.4, J14.4, Q5.2, R19.1
- removed net SCL3: J16.4, J17.4, J19.4, Q7.2, R27.1
- removed net SCL4: J21.4, J22.4, J24.4, Q9.2, R35.1
- removed net SCL5: J26.4, J27.4, J29.4, Q11.2, R43.1
- removed net SDA1: J6.3, J7.3, J9.3, Q4.2, R12.1
- removed net SDA2: J11.3, J12.3, J14.3, Q6.2, R21.1
- removed net SDA3: J16.3, J17.3, J19.3, Q8.2, R29.1
- removed net SDA4: J21.3, J22.3, J24.3, Q10.2, R37.1
- removed net SDA5: J26.3, J27.3, J29.3, Q12.2, R45.1
Routing:
- net 3.3V5: track 114.4 -> 0.00 mm, vias 3 -> 0
- net 3.3V3: track 114.4 -> 0.00 mm, vias 3 -> 0
- net 3.3V2: track 114.4 -> 0.00 mm, vias 3 -> 0
- net 3.3V1: track 114.4 -> 0.00 mm, vias 3 -> 0
- net 3.3V4: track 114.4 -> 0.00 mm, vias 3 -> 0
- net 5V5: track 112.5 -> 0.00 mm, vias 4 -> 0
- net 5V1: track 112.5 -> 0.00 mm, vias 4 -> 0
- net 5V4: track 112.5 -> 0.00 mm, vias 4 -> 0
- net 5V3: track 112.5 -> 0.00 mm, vias 4 -> 0
- net 5V2: track 112.5 -> 0.00 mm, vias 4 -> 0
- net SCL2: track 62.6 -> 0.00 mm, vias 3 -> 0
- net SCL3: track 62.6 -> 0.00 mm, vias 3 -> 0
- net SCL4: track 62.6 -> 0.00 mm, vias 3 -> 0
- net SCL5: track 62.6 -> 0.00 mm, vias 3 -> 0
- net SCL1: track 62.6 -> 0.00 mm, vias 3 -> 0
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- removed copper zone on layer 1, net GND1
- removed copper zone on layer 16, net GND1
- removed copper zone on layer 1, net GND2
- removed copper zone on layer 16, net GND2
- removed copper zone on layer 1, net GND3
- removed copper zone on layer 16, net GND3
- removed copper zone on layer 1, net GND4
- removed copper zone on layer 16, net GND4
- removed copper zone on layer 1, net GND5
- removed copper zone on layer 16, net GND5
Other:
- board size 152.7 x 152.4 mm -> 66 x 45.7 mm
- board text added: "NPoole"
- board text removed: "v-score"
