File: Hardware/qwiic_blower.sch (EAGLE design)
At the start: 33 parts, among them J1 QWIIC_RIGHT_ANGLE, J2 QWIIC_RIGHT_ANGLE, J3 AVR_SPI_PROG_3X2NS, Q2 310mA/60V/1.6Ω, Q3 310mA/60V/1.6Ω, U1 ATtiny841, U3 PAM2401, Y2 16MHz

Commit message: V1 Docs and Housecleaning
Other:
- note added: "NPoole"
Changed lines of the file:
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@@
 <wire x1="147.32" y1="96.52" x2="248.92" y2="96.52" width="0.2032" layer="97" style="longdash"/>
 <text x="43.18" y="33.02" size="2.54" layer="94" font="vector" align="center">Power LED</text>
+<text x="165.862" y="11.176" size="2.54" layer="94">NPoole</text>
 </plain>
 <instances>
